Commit message: UPDATE-- New URDF
updated urdf for Kassel

File: docker/abb_crb15000_dual_support/urdf/abb_crb15000_dual_cell.xacro (robot description, xacro)
@@ -13,5 +13,5 @@
     <parent link="world" />
     <child link = "robotB_base_link" />
-    <origin xyz="1.20434792	0.00855868803	0.00636037738" rpy="-0.00100184180	0.00949131399	-3.13337030"/>
+    <origin xyz="1.212360107012198	-0.014652473443031614	-0.002578851287850591" rpy="0.0011315789942580382	0.0.0015785551488194651	3.1324382669315396"/>
   </joint>
 </robot>

Commit message: update moveit package

File: docker/abb_crb15000_dual_support/urdf/abb_crb15000_dual_cell.xacro (robot description, xacro)
@@ -13,5 +13,5 @@
     <parent link="world" />
     <child link = "robotB_base_link" />
-    <origin xyz="1.212360107012198	-0.014652473443031614	-0.002578851287850591" rpy="0.0011315789942580382	0.0.0015785551488194651	3.1324382669315396"/>
+    <origin xyz="1.212360107012198	-0.014652473443031614	-0.002578851287850591" rpy="0.0011315789942580382	0.0015785551488194651	3.1324382669315396"/>
   </joint>
 </robot>

File: docker/abb_crb15000_dual_support/urdf/crb15000_5_95_macro.xacro (robot description, xacro)
@@ -137,5 +137,5 @@
       <parent link="${prefix}link_5"/>
       <child link="${prefix}link_6"/>
-      <limit effort="0" lower="${radians(-265)}" upper="${radians(265)}" velocity="${radians(200)}"/>
+      <limit effort="0" lower="${radians(-180)}" upper="${radians(180)}" velocity="${radians(200)}"/>
     </joint>
     <!-- end of joint list -->
